File: P2/Untitled.sch (KiCad schematic (older format))
At the start: 3 parts

Commit message: Additions 06062017
Parts:
- added C?: 10 uF, symbol C
- added C?: 0.1 uF, symbol C
- added U?: LTC6655-1.25, TO_SOT_Packages_SMD:SOT-23-5, symbol LTC6655-1.25
- TH?: value Thermistor 10k -> Thermistor1 10k
Connections:
- net labels added: ADC
- wire segments 4 -> 7
Other:
- moved on the sheet: R?, TH?, U?
Changed lines of the file:
@@
 LIBS:valves
 LIBS:opa189_ti
+LIBS:Untitled-cache
 EELAYER 25 0
 EELAYER END
@@
 L OPA189_TI U?
 U 1 1 5A20A66A
-P 4300 5450
-F 0 "U?" H 2750 9250 60  0000 C CNN
-F 1 "OPA189_TI" H 2850 8750 60  0000 C CNN
-F 2 "" H 4300 5450 60  0001 C CNN
-F 3 "" H 4300 5450 60  0001 C CNN
-	1    4300 5450
+P 5650 6300
+F 0 "U?" H 4100 10100 60  0000 C CNN
+F 1 "OPA189_TI" H 4200 9600 60  0000 C CNN
+F 2 "" H 5650 6300 60  0001 C CNN
+F 3 "" H 5650 6300 60  0001 C CNN
+	1    5650 6300
 	1    0    0    -1
 $EndComp
@@
 L Thermistor TH?
 U 1 1 5A20A771
-P 2550 1200
-F 0 "TH?" V 2650 1250 50  0000 C CNN
-F 1 "Thermistor 10k" V 2450 1200 50  0000 C BNN
-F 2 "" H 2550 1200 50  0001 C CNN
-F 3 "" H 2550 1200 50  0001 C CNN
-	1    2550 1200
+P 3900 2050
+F 0 "TH?" V 4000 2100 50  0000 C CNN
+F 1 "Thermistor1 10k" V 3800 2050 50  0000 C BNN
+F 2 "" H 3900 2050 50  0001 C CNN
+F 3 "" H 3900 2050 50  0001 C CNN
+	1    3900 2050
 	0    1    1    0
 $EndComp
 Wire Wire Line
-	2750 1200 3200 1200
+	4100 2050 4550 2050
 Wire Wire Line
-	3200 1200 3200 1850
+	4550 2050 4550 2700
 Wire Wire Line
-	2350 1200 2000 1200
+	3700 2050 3350 2050
 Wire Wire Line
-	2000 1200 2000 1750
+	3350 2050 3350 2600
 $Comp
 L GNDA #PWR01
 U 1 1 5A20A800
-P 2000 2050
-F 0 "#PWR01" H 2000 1800 50  0001 C CNN
-F 1 "GNDA" H 2000 1900 50  0000 C CNN
-F 2 "" H 2000 2050 50  0001 C CNN
-F 3 "" H 2000 2050 50  0001 C CNN
-	1    2000 2050
+P 3350 2900
+F 0 "#PWR01" H 3350 2650 50  0001 C CNN
+F 1 "GNDA" H 3350 2750 50  0000 C CNN
+F 2 "" H 3350 2900 50  0001 C CNN
+F 3 "" H 3350 2900 50  0001 C CNN
+	1    3350 2900
 	1    0    0    -1
 $EndComp
@@
 L R R?
 U 1 1 5A20A81C
-P 1850 1750
-F 0 "R?" V 1930 1750 50  0000 C CNN
-F 1 "10 k" V 1850 1750 50  0000 C CNN
-F 2 "" V 1780 1750 50  0001 C CNN
-F 3 "" H 1850 1750 50  0001 C CNN
-	1    1850 1750
+P 3200 2600
+F 0 "R?" V 3280 2600 50  0000 C CNN
+F 1 "10 k" V 3200 2600 50  0000 C CNN
+F 2 "" V 3130 2600 50  0001 C CNN
+F 3 "" H 3200 2600 50  0001 C CNN
+	1    3200 2600
 	0    1    1    0
 $EndComp
+$Comp
+L LTC6655-1.25 U?
+U 1 1 5A2837CC
+P 2550 2700
+F 0 "U?" H 2300 2900 50  0000 L CNN
+F 1 "LTC6655-1.25" H 3150 2900 50  0000 R CNN
+F 2 "TO_SOT_Packages_SMD:SOT-23-5" H 3200 2450 50  0001 C CIN
+F 3 "" H 2550 2700 50  0000 C CNN
+	1    2550 2700
+	1    0    0    -1
+$EndComp
+Wire Wire Line
+	2950 2600 3100 2600
+Connection ~ 3050 2600
+Wire Wire Line
+	2950 2600 2950 2800
+$Comp
+L C C?
+U 1 1 5A283EBF
+P 3050 2750
+F 0 "C?" H 3075 2850 50  0000 L CNN
+F 1 "10 uF" H 3075 2650 50  0000 L CNN
+F 2 "" H 3088 2600 50  0001 C CNN
+F 3 "" H 3050 2750 50  0001 C CNN
+	1    3050 2750
+	1    0    0    -1
+$EndComp
+$Comp
+L GNDA #PWR?
+U 1 1 5A283FC9
+P 3050 2900
+F 0 "#PWR?" H 3050 2650 50  0001 C CNN
+F 1 "GNDA" H 3050 2750 50  0000 C CNN
+F 2 "" H 3050 2900 50  0001 C CNN
+F 3 "" H 3050 2900 50  0001 C CNN
+	1    3050 2900
+	1    0    0    -1
+$EndComp
+$Comp
+L GNDA #PWR?
+U 1 1 5A284003
+P 2150 2800
+F 0 "#PWR?" H 2150 2550 50  0001 C CNN
+F 1 "GNDA" H 2150 2650 50  0000 C CNN
+F 2 "" H 2150 2800 50  0001 C CNN
+F 3 "" H 2150 2800 50  0001 C CNN
+	1    2150 2800
+	1    0    0    -1
+$EndComp
+$Comp
+L C C?
+U 1 1 5A28410D
+P 2150 2700
+F 0 "C?" H 2175 2800 50  0000 L CNN
+F 1 "0.1 uF" H 2175 2600 50  0000 L CNN
+F 2 "" H 2188 2550 50  0001 C CNN
+F 3 "" H 2150 2700 50  0001 C CNN
+	1    2150 2700
+	1    0    0    -1
+$EndComp
+Connection ~ 3350 2600
+Connection ~ 4550 2700
+Connection ~ 2150 2600
+Wire Wire Line
+	4550 2700 4900 2700
+Text HLabel 4900 2700 2    60   Output ~ 0
+ADC
 $EndSCHEMATC
